Commit message: Fixed pinocchio_utils

File: src/assets/urdf/indy7_v2/indy7_v2/model.urdf (robot description, URDF)
Before this commit: robot indy, 8 links, 7 joints
Joints:
- removed joint tcp
- added joint indy0_joint_tcp: type fixed, parent indy0_link6, child tcp, origin xyz=0.0 0.0 0.06 rpy=0.0 0.0 0.0, axis 0.0 0.0 1.0
